Commit message: successfully train with go2_d1 config

File: go2_d1_description/go2_d1_description/urdf/go2_d1.urdf (robot description, URDF)
Before this commit: robot go2_description, 37 links, 36 joints
Links:
- added link RR_foot, mass 0.04; collision sphere radius=0.022; visual mesh filename=/home/adam/ChongQing/Go2Arm_Lab/go2_d1_description/go2_d1_d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
Joints:
- added joint RR_foot_joint: type fixed, parent RR_calf, child RR_foot, origin xyz=0 0 -0.213 rpy=0 0 0, axis 0 0 0
